File: ConceptionPCB_Projet_PAZ/Projet_PAZ/Capteur_humidite_pulsation_temperature.kicad_sch (KiCad schematic)
At the start: 9 parts, among them Q1 BPW85

Commit message: Add files via upload
Parts:
- H7, H8: footprint MountingHole:MountingHole_3.2mm_M3_DIN965_Pad -> MesEmpreintes:ConnexionPAZ
Changed lines of the file:
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@@
       (effects (font (size 1.27 1.27)))
     )
-    (property "Footprint" "MountingHole:MountingHole_3.2mm_M3_DIN965_Pad" (at 130.81 111.125 0)
+    (property "Footprint" "MesEmpreintes:ConnexionPAZ" (at 130.81 111.125 0)
       (effects (font (size 1.27 1.27)) hide)
     )
@@
       (effects (font (size 1.27 1.27)))
     )
-    (property "Footprint" "MountingHole:MountingHole_3.2mm_M3_DIN965_Pad" (at 109.855 111.125 0)
-      (effects (font (size 1.27 1.27)) hide)
-    )
+    (property "Footprint" "MesEmpreintes:ConnexionPAZ" (at 109.855 111.125 0)
+      (effects (font (size 1.27 1.27)) hide)
+    )
