File: ConceptionPCB_Projet_PAZ/Projet_PAZ/Projet_PAZ.kicad_pcb (KiCad board)
At the start: 2 copper layers, 52 parts, among them IC1 STM32L412KBT6, J2 Conn_02x07_Odd_Even, J3 XT60-M, Q1 BPW85, Q3 2N2905A, U1 BU33SD5WG-TR

Commit message: Add files via upload
Parts:
- added H1: MountingHole_Pad, MountingHole:MountingHole_2.5mm_Pad, F.Cu at (167.8, 70.8)
- added H11: MountingHole_Pad, MountingHole:MountingHole_2.5mm_Pad, F.Cu at (207.8, 70.8)
- added H12: MountingHole_Pad, MountingHole:MountingHole_2.5mm_Pad, F.Cu at (207.8, 81.8)
- added H13: MountingHole_Pad, MountingHole:MountingHole_2.5mm_Pad, F.Cu at (222.8, 70.8)
- added H14: MountingHole_Pad, MountingHole:MountingHole_2.5mm_Pad, F.Cu at (222.8, 81.8)
- added H15: MountingHole_Pad, MountingHole:MountingHole_2.5mm_Pad, F.Cu at (191.6, 105.0)
- added H16: MountingHole_Pad, MountingHole:MountingHole_2.5mm_Pad, F.Cu at (191.6, 90.0)
- added H17: MountingHole_Pad, MountingHole:MountingHole_2.5mm_Pad, F.Cu at (225.6, 90.0)
- added H18: MountingHole_Pad, MountingHole:MountingHole_2.5mm_Pad, F.Cu at (225.6, 105.0)
- added H3: MountingHole_Pad, MountingHole:MountingHole_2.5mm_Pad, F.Cu at (167.8, 81.8)
- added H4: MountingHole_Pad, MountingHole:MountingHole_2.5mm_Pad, F.Cu at (182.8, 70.8)
- added H6: MountingHole_Pad, MountingHole:MountingHole_2.5mm_Pad, F.Cu at (182.8, 81.8)
- H7, H8: footprint MountingHole:MountingHole_3.2mm_M3_DIN965_Pad -> MesEmpreintes:ConnexionPAZ
- moved R3 163.7 mm to (196.1, 96.1), turned to -90 degrees
- moved C7 162.1 mm to (222.9, 113.4)
- moved R11 156.5 mm to (219.4, 113.4)
- moved R17 150.9 mm to (215.9, 113.4)
- moved C6 137.9 mm to (190.9, 113.4), turned to 180 degrees
- moved R4 137.4 mm to (194.4, 113.4)
- moved R16 137.2 mm to (197.9, 113.4)
- moved R2 130.4 mm to (162.9, 111.0)
- moved C5 130.3 mm to (203.4, 73.1), turned to -90 degrees
- moved D3 129.2 mm to (158.9, 111.0), turned to 180 degrees
- moved H10 127.7 mm to (229.9, 66.1), turned to 0 degrees
- moved C12 125.8 mm to (141.8, 109.9), turned to 90 degrees
- moved C18 125.7 mm to (143.8, 115.1), turned to -90 degrees
- moved C17 124.0 mm to (143.8, 109.9), turned to -90 degrees
- moved C16 122.7 mm to (139.8, 109.9), turned to 90 degrees
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Routing:
- net GND: track 0.00 -> 769.7 mm, vias 0 -> 9
- net +3.3V: track 0.00 -> 324.6 mm, vias 0 -> 4
- net +5V: track 0.00 -> 207.3 mm, vias 0 -> 2
- net SYS_SWDIO: track 0.00 -> 94.2 mm, vias 0 -> 2
- net I2C1_SCL: track 0.00 -> 86.9 mm
- net USART2_RX: track 0.00 -> 82.7 mm, vias 0 -> 2
- net SYS_SWCLK: track 0.00 -> 79.1 mm, vias 0 -> 2
- net Moist: track 0.00 -> 78.6 mm, vias 0 -> 2
- net USART2_TX: track 0.00 -> 78.1 mm, vias 0 -> 2
- net D_B2: track 0.00 -> 76.7 mm, vias 0 -> 2
- net I2C3_SCL: track 0.00 -> 74.8 mm, vias 0 -> 1
- net I2C1_SDA: track 0.00 -> 66.7 mm
- net NRST: track 0.00 -> 66.5 mm, vias 0 -> 2
- net I2C3_SDA: track 0.00 -> 65.8 mm
- net Buzzer: track 0.00 -> 62.4 mm, vias 0 -> 2
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- added copper zone on B.Cu, net GND
- added copper zone on F.Cu, net GND
Other:
- board outline added: 148.9 x 68.8 mm
- board text added: "+3.3V"
- board text added: "+5V"
- board text added: "Alim. Générale"
- board text added: "Bouton n°1"
- board text added: "Bouton n°2"
- board text added: "Buzzer"
- board text added: "Capteur cardiaque"
- board text added: "Capteur d'humidité"
- board text added: "Capteur de température"
- board text added: "Connecteur Ecran OLED"
- board text added: "Connecteur SWD"
- board text added: "Données analogiques"
- board text added: "Données numériques"
- board text added: "Led de contrôle STM32"
- board text added: "Led seuil +3.3V"
- board text added: "Support Ecran OLED"
- board text added: "µC STM32"
