File: ConceptionPCB_Projet_PAZ/Projet_PAZ/Projet_PAZ.kicad_sch (KiCad schematic)
At the start: 40 parts, among them J1 Conn_01x03, J13 Conn_01x02, J2 Conn_01x03, J7 Conn_01x03, J9 Conn_02x07_Odd_Even, SW1 SW_SPDT, U2 STM32L021K4Tx, U4 BU33SD5WG-TR

Commit message: Add files via upload
Parts:
- removed J7: Conn_01x03, symbol Connector_Generic:Conn_01x03
Connections:
- no-connect marks 16 -> 18
Changed lines of the file:
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@@
   (no_connect (at 81.28 122.555))
   (no_connect (at 38.1 35.56))
+  (no_connect (at 167.64 127.635))
   (no_connect (at 81.28 111.125))
   (no_connect (at 98.425 168.275))
@@
   (no_connect (at 254.635 102.235))
   (no_connect (at 239.395 102.235))
+  (no_connect (at 167.64 130.175))
   (no_connect (at 98.425 178.435))
   (no_connect (at 81.28 126.365))
@@
         )
       )
-    )
-  )
-  (symbol (lib_id "Connector_Generic:Conn_01x03") (at 278.765 173.355 0) (unit 1)
-    (in_bom yes) (on_board yes) (dnp no)
-    (property "Reference" "J7" (at 281.305 172.085 0)
-      (effects (font (size 1.27 1.27)) (justify left))
-    )
-    (property "Value" "Conn_01x03" (at 281.305 174.625 0)
-      (effects (font (size 1.27 1.27)) (justify left))
-    )
-    (property "Footprint" "" (at 278.765 173.355 0)
-      (effects (font (size 1.27 1.27)) hide)
-    )
-    (property "Datasheet" "~" (at 278.765 173.355 0)
-      (effects (font (size 1.27 1.27)) hide)
-    )
-    (pin "1")
-    (pin "2")
-    (pin "3")
-    (instances
-      (project "Projet_PAZ"
-        (path "/2ce892fe-c082-4bae-b2dd-3c3e6d69cf95"
-          (reference "J7") (unit 1)
-        )
-      )

Commit message: Add files via upload
Parts:
- removed C7: 100nF, symbol Device:C_Small
- removed D4: Statut du microcontrôleur, LED_SMD:LED_0603_1608Metric_Pad1.05x0.95mm_HandSolder, symbol Device:LED_Small
- removed R1: 10k, symbol Device:R_Small
- removed R2: 1k, Resistor_SMD:R_0603_1608Metric_Pad0.98x0.95mm_HandSolder, symbol Device:R_Small
- removed U2: STM32L021K4Tx, Package_QFP:LQFP-32_7x7mm_P0.8mm, symbol MCU_ST_STM32L0:STM32L021K4Tx
- removed U3: ~, symbol MesSymboles:INT028ATFT
- added C13: 100nF, symbol Device:C_Small
- added C14, C15: C_Small, symbol Device:C_Small
- added D1: Statut du microcontrôleur, LED_SMD:LED_0603_1608Metric_Pad1.05x0.95mm_HandSolder, symbol Device:LED_Small
- added H5, H6: MountingHole_Pad, MountingHole:MountingHole_3.2mm_M3_DIN965_Pad, symbol Mechanical:MountingHole_Pad
- added IC1: STM32L412KBT6, QFP80P900X900X160-32N, symbol STM32L412KBT6:STM32L412KBT6
- added J3: Conn_01x04, symbol Connector_Generic:Conn_01x04
- added R10: 1k, Resistor_SMD:R_0603_1608Metric_Pad0.98x0.95mm_HandSolder, symbol Device:R_Small
- added R9: 10k, symbol Device:R_Small
- added U1, U3: ~, symbol MesSymboles:MDOB128064WV-YBI
Connections:
- net +3.3V: now also IC1.1 (VDD_1), IC1.17 (VDD_2)
- net +3.3VA: now also IC1.5 (VDDA/VREF+)
- net +5V: now also J3.3 (Pin_3)
- net D_B1: now also IC1.2 (PC14-OSC32_IN)
- net D_B2: now also IC1.3 (PC15-OSC32_OUT)
- net GND: now also C13.1, C14.2, C15.2, H5.1, H6.1, IC1.16 (VSS_1), IC1.32 (VSS_2), J3.4 (Pin_4), R10.2, R9.1, U1.2 (GND), U3.2 (GND)
- net LED_STATUS: now also D1.2 (A), IC1.22 (PA12)
- net NRST: now also C13.2, IC1.4 (NRST)
- net Puls: now also IC1.10 (PA4)
- net SYS_SWCLK: now also IC1.24 (PA14)
- net SYS_SWDIO: now also IC1.23 (PA13)
- net Temp: now also IC1.7 (PA1)
- net USART2_RX: now also IC1.9 (PA3)
- net USART2_TX: now also IC1.8 (PA2)
- new net: C14.1, U1.1 (VCC)
- new net: IC1.31 (PH3-BOOT0), R9.2
- new net: C15.1, U3.1 (VCC)
- new net: D1.1 (K), R10.1
- new net Buzzer: IC1.11 (PA5), J3.1 (Pin_1)
- new net I2C1_SCL: IC1.19 (PA9), U1.13 (SCL)
- new net I2C1_SDA: IC1.20 (PA10), U1.14 (SDA)
- new net I2C3_SCL: IC1.13 (PA7), U3.13 (SCL)
- new net I2C3_SDA: IC1.27 (PB4), U3.14 (SDA)
- no-connect marks 18 -> 22
Other:
- note added: "Ecran Oled"
- note removed: "Ecran TFT"
- moved on the sheet: C1, C12, C2, C3, C4, C5, C6, C8, C9, D5, D6, D7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

Commit message: Add files via upload
Parts:
- removed H2, H5: MountingHole_Pad, MountingHole:MountingHole_3.2mm_M3_DIN965_Pad, symbol Mechanical:MountingHole_Pad
- removed J1, J2: Conn_01x03, symbol Connector_Generic:Conn_01x03
- removed J3: Conn_01x04, symbol Connector_Generic:Conn_01x04
- removed U3: ~, symbol MesSymboles:MDOB128064WV-YBI
- added H7, H8: MountingHole_Pad, MountingHole:MountingHole_3.2mm_M3_DIN965_Pad, symbol Mechanical:MountingHole_Pad
- added J1: Conn_01x02, symbol Connector_Generic:Conn_01x02
- added Q1: Q_Photo_NPN, symbol Device:Q_Photo_NPN
- added Q3: 2N2219, Package_TO_SOT_THT:TO-39-3, symbol Transistor_BJT:2N2219
- added R1: 1M, symbol Device:R
- added R11, R12: R_Small, symbol Device:R_Small
- added R2: 10k, Resistor_SMD:R_0805_2012Metric, symbol Device:R
- added RT1: B57164K0472J000, B57164K_K164, symbol B57164K0472J000:B57164K0472J000
- added U2: ~, symbol MesSymboles:MDOB128064WV-YBI
- C14, C15: value C_Small -> 1µF
- R10, R3, R4: value 1k -> 470
Connections:
- net +3.3V: now also J1.1 (Pin_1), R1.2
- net +5V: now also R12.1, R2.1
- net Buzzer: now also IC1.26 (PB3), R11.1
- net D_B1: now also IC1.14 (PB0); no longer IC1.2 (PC14-OSC32_IN)
- net D_B2: now also IC1.15 (PB1); no longer IC1.3 (PC15-OSC32_OUT)
- net GND: now also H7.1, Q1.2 (E), Q3.1 (E), RT1.2, U2.2 (GND)
- net I2C1_SCL: now also U1.3 (SCL); no longer U1.13 (SCL)
- net I2C1_SDA: now also U1.4 (SDA); no longer U1.14 (SDA)
- net I2C3_SCL: now also U2.3 (SCL)
- net I2C3_SDA: now also U2.4 (SDA)
- net Puls: now also Q1.1 (C), R12.2
- net Temp: now also R2.2, RT1.1
- net at C15.1: now also U2.1 (VCC)
- new net: J1.2 (Pin_2), Q3.3 (C)
- new net: Q3.2 (B), R11.2
- new net Moist: H8.1, R1.1
- no-connect marks 22 -> 20
Other:
- note added: "Buzzer"
- note added: "Capteur d'humidité"
- note added: "Capteur de pulsation"
- note added: "Capteur de températeur"
- note added: "Il manque la photo diode + resistance"
- note removed: "Connecteurs d'entrées/sorties"
- moved on the sheet: C1, C10, C11, C12, C13, C14, C15, C2, C3, C4, C5, C6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

Commit message: Add files via upload
Parts:
- removed C12: 10µ, Capacitor_SMD:C_0805_2012Metric, symbol Device:C
- removed D6: D, Diode_SMD:D_0805_2012Metric, symbol Device:D
- removed IC1: STM32L412KBT6, QFP80P900X900X160-32N, symbol STM32L412KBT6:STM32L412KBT6
- removed Q1: Q_Photo_NPN, symbol Device:Q_Photo_NPN
- removed R12: R_Small, symbol Device:R_Small
- added C7: 1µF, Capacitor_SMD:C_0603_1608Metric_Pad1.08x0.95mm_HandSolder, symbol Device:C_Small
- added D2: D_Small, LED_SMD:LED_0603_1608Metric_Pad1.05x0.95mm_HandSolder, symbol Device:D_Small
- added D4: IR204A, LED_THT:LED_D3.0mm_IRBlack, symbol LED:IR204A
- added IC2: STM32L412KBT6, MesEmpreintes:QFP80P900X900X160-32N, symbol STM32L412KBT6:STM32L412KBT6
- added Q5: Q_Photo_NPN, symbol Device:Q_Photo_NPN
- added R15: 10k, Resistor_SMD:R_0603_1608Metric_Pad0.98x0.95mm_HandSolder, symbol Device:R
- added R16: 320, Resistor_SMD:R_0603_1608Metric_Pad0.98x0.95mm_HandSolder, symbol Device:R
- C10, C11: footprint Capacitor_SMD:C_0805_2012Metric -> Capacitor_SMD:C_0603_1608Metric_Pad1.08x0.95mm_HandSolder
- C13, C14: footprint (none) -> Capacitor_SMD:C_0603_1608Metric_Pad1.08x0.95mm_HandSolder
- C15: value 1µF -> 10µ; footprint (none) -> Capacitor_SMD:C_0603_1608Metric_Pad1.08x0.95mm_HandSolder
- R1, R9: footprint (none) -> Resistor_SMD:R_0603_1608Metric_Pad0.98x0.95mm_HandSolder
- R11: value R_Small -> 220; footprint (none) -> Resistor_SMD:R_0603_1608Metric_Pad0.98x0.95mm_HandSolder
- R2: footprint Resistor_SMD:R_0805_2012Metric -> Resistor_SMD:R_0603_1608Metric_Pad0.98x0.95mm_HandSolder
- R4: value 470 -> ohm
- R5, R6: value 150 -> ohm; footprint Resistor_SMD:R_0805_2012Metric -> Resistor_SMD:R_0603_1608Metric_Pad0.98x0.95mm_HandSolder
- R7, R8: value 10k -> ohm; footprint Resistor_SMD:R_0805_2012Metric -> Resistor_SMD:R_0603_1608Metric_Pad0.98x0.95mm_HandSolder
- RT1: footprint B57164K_K164 -> MesEmpreintes:B57164K_K164
- S1, S2: footprint TL1100F160Q:SW_TL1100F160Q -> MesEmpreintes:SW_TL1100F160Q
Connections:
- net +3.3V: now also C14.1, R2.1, U1.1 (VCC), U2.1 (VCC), C7.1, IC2.1 (VDD_1), IC2.17 (VDD_2)
- net +3.3VA: now also IC2.5 (VDDA/VREF+)
- net +5V: now also C15.2, D2.1 (K), R15.1, R16.2; no longer R2.1
- net Buzzer: now also IC2.11 (PA5), IC2.26 (PB3)
- net D_B1: now also IC2.14 (PB0)
- net D_B2: now also IC2.15 (PB1)
- net GND: now also C15.1, C7.2, D2.2 (A), D4.1 (K), IC2.16 (VSS_1), IC2.32 (VSS_2), Q5.2 (E); no longer C15.2
- net I2C1_SCL: now also IC2.19 (PA9)
- net I2C1_SDA: now also IC2.20 (PA10)
- net I2C3_SCL: now also IC2.13 (PA7)
- net I2C3_SDA: now also IC2.27 (PB4)
- net LED_STATUS: now also IC2.22 (PA12)
- net Moist: now also IC2.12 (PA6)
- net NRST: now also IC2.4 (NRST)
- net Puls: now also IC2.10 (PA4), Q5.1 (C), R15.2
- net SYS_SWCLK: now also IC2.24 (PA14)
- net SYS_SWDIO: now also IC2.23 (PA13)
- net Temp: now also IC2.7 (PA1)
- net USART2_RX: now also IC2.9 (PA3)
- net USART2_TX: now also IC2.8 (PA2)
- net at R9.2: now also IC2.31 (PH3-BOOT0)
- new net: D4.2 (A), R16.1
- no-connect marks 20 -> 19
Other:
- note added: "Capteur de température"
- note removed: "Capteur de températeur"
- note removed: "Il manque la photo diode + resistance"
- moved on the sheet: C1, C13, C14, C2, C3, C4, C5, C6, C8, C9, D1, D5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

Commit message: Add files via upload
Parts:
- removed SW1: SW_SPDT, Interrupteur_a_glissiere:OS102011MS2QS1, symbol Switch:SW_SPDT
- added S3: KSS221G, MesEmpreintes:KSS221G, symbol KSS221G:KSS221G
Connections:
- net +3.3V: now also R15.1, R16.2
- net +5V: now also S3.2; no longer R15.1, R16.2
- net at J13.2 (Pin_2): now also S3.1
Other:
- moved on the sheet: C8, C9, D5, R3, U4

Commit message: Add files via upload
Parts:
- removed C1, C14, C7: 1µF, Capacitor_SMD:C_0603_1608Metric_Pad1.08x0.95mm_HandSolder, symbol Device:C_Small
- removed C10, C11: 100n, Capacitor_SMD:C_0603_1608Metric_Pad1.08x0.95mm_HandSolder, symbol Device:C
- removed C13, C3, C4, C5: 100nF, Capacitor_SMD:C_0603_1608Metric_Pad1.08x0.95mm_HandSolder, symbol Device:C_Small
- removed C15: 10µ, Capacitor_SMD:C_0603_1608Metric_Pad1.08x0.95mm_HandSolder, symbol Device:C_Small
- removed C2: 10nF, Capacitor_SMD:C_0603_1608Metric_Pad1.08x0.95mm_HandSolder, symbol Device:C_Small
- removed C6: 4,7µF, Capacitor_SMD:C_0603_1608Metric_Pad1.08x0.95mm_HandSolder, symbol Device:C_Small
- removed D1: Statut du microcontrôleur, LED_SMD:LED_0603_1608Metric_Pad1.05x0.95mm_HandSolder, symbol Device:LED_Small
- removed D2: D_Small, LED_SMD:LED_0603_1608Metric_Pad1.05x0.95mm_HandSolder, symbol Device:D_Small
- removed D4: IR204A, LED_THT:LED_D3.0mm_IRBlack, symbol LED:IR204A
- removed D5: Témoin d'alimentation Microcontrôleur STM32, LED_SMD:LED_0603_1608Metric_Pad1.05x0.95mm_HandSolder, symbol Device:LED_Small
- removed H1, H3, H4, H6, H7, H8: MountingHole_Pad, MountingHole:MountingHole_3.2mm_M3_DIN965_Pad, symbol Mechanical:MountingHole_Pad
- removed IC2: STM32L412KBT6, MesEmpreintes:QFP80P900X900X160-32N, symbol STM32L412KBT6:STM32L412KBT6
- removed J1: Conn_01x02, symbol Connector_Generic:Conn_01x02
- removed J13: Conn_01x02, Connecteur_alimentation:connecteur, symbol Connector_Generic:Conn_01x02
- removed J9: Conn_02x07_Odd_Even, Connector_PinHeader_1.27mm:PinHeader_2x07_P1.27mm_Vertical_SMD, symbol Connector_Generic:Conn_02x07_Odd_Even
- removed L1: 39nH, Inductor_SMD:L_0603_1608Metric_Pad1.05x0.95mm_HandSolder, symbol Device:L_Small
- removed Q3: 2N2219, Package_TO_SOT_THT:TO-39-3, symbol Transistor_BJT:2N2219
- removed Q5: Q_Photo_NPN, symbol Device:Q_Photo_NPN
- removed R1: 1M, Resistor_SMD:R_0603_1608Metric_Pad0.98x0.95mm_HandSolder, symbol Device:R
- removed R10, R3: 470, Resistor_SMD:R_0603_1608Metric_Pad0.98x0.95mm_HandSolder, symbol Device:R_Small
- removed R11: 220, Resistor_SMD:R_0603_1608Metric_Pad0.98x0.95mm_HandSolder, symbol Device:R_Small
- removed R15, R2: 10k, Resistor_SMD:R_0603_1608Metric_Pad0.98x0.95mm_HandSolder, symbol Device:R
- removed R16: 320, Resistor_SMD:R_0603_1608Metric_Pad0.98x0.95mm_HandSolder, symbol Device:R
- removed R4: ohm, Resistor_SMD:R_0603_1608Metric_Pad0.98x0.95mm_HandSolder, symbol Device:R_Small
- removed R5, R6, R7, R8: ohm, Resistor_SMD:R_0603_1608Metric_Pad0.98x0.95mm_HandSolder, symbol Device:R
- removed R9: 10k, Resistor_SMD:R_0603_1608Metric_Pad0.98x0.95mm_HandSolder, symbol Device:R_Small
- removed RT1: B57164K0472J000, MesEmpreintes:B57164K_K164, symbol B57164K0472J000:B57164K0472J000
- removed S1, S2: TL1100F160Q, MesEmpreintes:SW_TL1100F160Q, symbol TL1100F160Q:TL1100F160Q
- removed S3: KSS221G, MesEmpreintes:KSS221G, symbol KSS221G:KSS221G
- removed U1, U2: ~, symbol MesSymboles:MDOB128064WV-YBI
- removed U4: BU33SD5WG-TR, Package_TO_SOT_SMD:SOT-23-5, symbol Regulator_Linear:MCP1802x-xx02xOT
- added C10: 1µF, Capacitor_SMD:C_0603_1608Metric_Pad1.08x0.95mm_HandSolder, symbol Device:C_Small
- added D2: Témoin d'alimentation général, LED_SMD:LED_0603_1608Metric_Pad1.05x0.95mm_HandSolder, symbol Device:LED_Small
- added D5: Diode_securitaire, Diode_SMD:D_0603_1608Metric_Pad1.05x0.95mm_HandSolder, symbol Device:D_Small
- added J3: XT60-M, MesEmpreintes:AMASS_XT60-M, symbol XT60-M:XT60-M
- added R5: ohm, Resistor_SMD:R_0603_1608Metric_Pad0.98x0.95mm_HandSolder, symbol Device:R_Small
- added R6: 470, Resistor_SMD:R_0603_1608Metric_Pad0.98x0.95mm_HandSolder, symbol Device:R_Small
- added S1: KSS221G, MesEmpreintes:KSS221G, symbol KSS221G:KSS221G
- added U1: BU33SD5WG-TR, Package_TO_SOT_SMD:SOT-23-5, symbol Regulator_Linear:MCP1802x-xx02xOT
- C8: value 1µF -> 10µ
- D7: value Témoin d'alimentation général -> Témoin d'alimentation Microcontrôleur STM32
Connections:
- net +3.3V: now also D7.2 (A), C10.1, U1.5 (VOUT); no longer C9.1
- net +5V: now also C8.2, C9.1, D5.1 (K), R5.2, S1.2, U1.1 (VIN), U1.3 (~{SHDN}); no longer C8.1
- net GND: now also C8.1, C10.2, D2.1 (K), D5.2 (A), J3.N (NEG), R6.2, U1.2 (GND); no longer C8.2, D7.1 (K)
- new net: D2.2 (A), R5.1
- new net: J3.P (POS), S1.1
- new net: D7.1 (K), R6.1
- no-connect marks 19 -> 0
Other:
- added sheet Boutons poussoirs (Boutons_poussoirs.kicad_sch)
- added sheet Buzzer (Buzzer.kicad_sch)
- added sheet Capteur d'humidité, de pulsation, de température (Capteur_humidite_pulsation_temperature.kicad_sch)
- added sheet Connecteur SWD (Connecteur_SWD.kicad_sch)
- added sheet Ecran Oled (Ecran_Oled.kicad_sch)
- added sheet Microcontrôleur STM32 (Microcontroleur_STM32.kicad_sch)
- added sheet Trou de fixation (Trou_de_fixation.kicad_sch)
- note removed: "Boutons poussoirs"
- note removed: "Buzzer"
- note removed: "Capteur d'humidité"
- note removed: "Capteur de pulsation"
- note removed: "Capteur de température"
- note removed: "Connecteur SWD"
- note removed: "Ecran Oled"
- note removed: "Microcontrôleur STM32"
- note removed: "Trous de fixation"

Commit message: Add files via upload
Changed lines of the file:
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@@
     (stroke (width 0) (type default))
   )
-  (wire (pts (xy 223.52 121.285) (xy 224.79 121.285))
+  (wire (pts (xy 222.885 131.445) (xy 224.155 131.445))
     (stroke (width 0) (type default))
   )
@@
     (stroke (width 0) (type default))
   )
-  (wire (pts (xy 223.52 130.81) (xy 224.79 130.81))
+  (wire (pts (xy 222.885 140.97) (xy 224.155 140.97))
     (stroke (width 0) (type default))
   )
@@
     (stroke (width 0) (type default))
   )
-  (wire (pts (xy 255.905 34.925) (xy 257.81 34.925))
+  (wire (pts (xy 255.27 40.005) (xy 257.175 40.005))
     (stroke (width 0) (type default))
   )
@@
     (stroke (width 0) (type default))
   )
-  (wire (pts (xy 223.52 117.475) (xy 224.79 117.475))
+  (wire (pts (xy 222.885 127.635) (xy 224.155 127.635))
     (stroke (width 0) (type default))
   )
@@
     (stroke (width 0) (type default))
   )
-  (wire (pts (xy 223.52 127) (xy 224.79 127))
+  (wire (pts (xy 222.885 137.16) (xy 224.155 137.16))
     (stroke (width 0) (type default))
   )
@@
     (stroke (width 0) (type default))
   )
-  (wire (pts (xy 255.905 39.37) (xy 257.81 39.37))
+  (wire (pts (xy 255.27 44.45) (xy 257.175 44.45))
     (stroke (width 0) (type default))
   )
@@
     (stroke (width 0) (type default))
   )
-  (wire (pts (xy 255.905 43.815) (xy 257.81 43.815))
+  (wire (pts (xy 255.27 48.895) (xy 257.175 48.895))
     (stroke (width 0) (type default))
   )
@@
     )
   )
-  (global_label "I2C1_SCL" (shape input) (at 223.52 127 180) (fields_autoplaced)
-    (effects (font (size 1.27 1.27)) (justify right))
-    (property "Intersheetrefs" "${INTERSHEET_REFS}" (at 211.7658 127 0)
+  (global_label "I2C1_SCL" (shape input) (at 222.885 137.16 180) (fields_autoplaced)
+    (effects (font (size 1.27 1.27)) (justify right))
+    (property "Intersheetrefs" "${INTERSHEET_REFS}" (at 211.1308 137.16 0)
       (effects (font (size 1.27 1.27)) (justify right) hide)
     )
@@
     )
   )
-  (global_label "I2C3_SCL" (shape input) (at 223.52 121.285 180) (fields_autoplaced)
-    (effects (font (size 1.27 1.27)) (justify right))
-    (property "Intersheetrefs" "${INTERSHEET_REFS}" (at 211.7658 121.285 0)
-      (effects (font (size 1.27 1.27)) (justify right) hide)
-    )
-  )
-  (global_label "I2C3_SDA" (shape input) (at 223.52 117.475 180) (fields_autoplaced)
-    (effects (font (size 1.27 1.27)) (justify right))
-    (property "Intersheetrefs" "${INTERSHEET_REFS}" (at 211.7053 117.475 0)
-      (effects (font (size 1.27 1.27)) (justify right) hide)
-    )
-  )
-  (global_label "Temp" (shape output) (at 257.81 39.37 0) (fields_autoplaced)
+  (global_label "I2C3_SCL" (shape input) (at 222.885 131.445 180) (fields_autoplaced)
+    (effects (font (size 1.27 1.27)) (justify right))
+    (property "Intersheetrefs" "${INTERSHEET_REFS}" (at 211.1308 131.445 0)
+      (effects (font (size 1.27 1.27)) (justify right) hide)
+    )
+  )
+  (global_label "I2C3_SDA" (shape input) (at 222.885 127.635 180) (fields_autoplaced)
+    (effects (font (size 1.27 1.27)) (justify right))
+    (property "Intersheetrefs" "${INTERSHEET_REFS}" (at 211.0703 127.635 0)
+      (effects (font (size 1.27 1.27)) (justify right) hide)
+    )
+  )
+  (global_label "Temp" (shape output) (at 257.175 44.45 0) (fields_autoplaced)
     (effects (font (size 1.27 1.27)) (justify left))
-    (property "Intersheetrefs" "${INTERSHEET_REFS}" (at 265.6937 39.37 0)
+    (property "Intersheetrefs" "${INTERSHEET_REFS}" (at 265.0587 44.45 0)
       (effects (font (size 1.27 1.27)) (justify left) hide)
     )
   )
-  (global_label "I2C1_SDA" (shape input) (at 223.52 130.81 180) (fields_autoplaced)
-    (effects (font (size 1.27 1.27)) (justify right))
-    (property "Intersheetrefs" "${INTERSHEET_REFS}" (at 211.7053 130.81 0)
+  (global_label "I2C1_SDA" (shape input) (at 222.885 140.97 180) (fields_autoplaced)
+    (effects (font (size 1.27 1.27)) (justify right))
+    (property "Intersheetrefs" "${INTERSHEET_REFS}" (at 211.0703 140.97 0)
       (effects (font (size 1.27 1.27)) (justify right) hide)
     )
@@
     )
   )
-  (global_label "Moist" (shape output) (at 257.81 43.815 0) (fields_autoplaced)
+  (global_label "Moist" (shape output) (at 257.175 48.895 0) (fields_autoplaced)
     (effects (font (size 1.27 1.27)) (justify left))
-    (property "Intersheetrefs" "${INTERSHEET_REFS}" (at 265.7542 43.815 0)
+    (property "Intersheetrefs" "${INTERSHEET_REFS}" (at 265.1192 48.895 0)
       (effects (font (size 1.27 1.27)) (justify left) hide)
     )
@@
     )
   )
-  (global_label "Puls" (shape output) (at 257.81 34.925 0) (fields_autoplaced)
+  (global_label "Puls" (shape output) (at 257.175 40.005 0) (fields_autoplaced)
     (effects (font (size 1.27 1.27)) (justify left))
-    (property "Intersheetrefs" "${INTERSHEET_REFS}" (at 264.9075 34.925 0)
+    (property "Intersheetrefs" "${INTERSHEET_REFS}" (at 264.2725 40.005 0)
       (effects (font (size 1.27 1.27)) (justify left) hide)
     )
@@
     )
   )
-  (sheet (at 224.79 113.665) (size 26.035 20.955)
+  (sheet (at 224.155 123.825) (size 26.035 20.955)
     (stroke (width 0.1524) (type solid))
     (fill (color 0 0 0 0.0000))
-    (property "Sheetname" "Ecran Oled" (at 226.695 113.03 0)
+    (property "Sheetname" "Ecran Oled" (at 226.06 123.19 0)
       (effects (font (size 2.54 2.54) bold) (justify left bottom))
     )
-    (property "Sheetfile" "Ecran_Oled.kicad_sch" (at 224.79 135.255 0)
+    (property "Sheetfile" "Ecran_Oled.kicad_sch" (at 224.155 145.415 0)
       (effects (font (size 1.27 1.27)) (justify left top))
     )
-    (pin "I2C3_SDA" input (at 224.79 117.475 180)
-      (effects (font (size 1.27 1.27)) (justify left))
-    )
-    (pin "I2C3_SCL" input (at 224.79 121.285 180)
-      (effects (font (size 1.27 1.27)) (justify left))
-    )
-    (pin "I2C1_SCL" input (at 224.79 127 180)
-      (effects (font (size 1.27 1.27)) (justify left))
-    )
-    (pin "I2C1_SDA" input (at 224.79 130.81 180)
+    (pin "I2C3_SDA" input (at 224.155 127.635 180)
+      (effects (font (size 1.27 1.27)) (justify left))
+    )
+    (pin "I2C3_SCL" input (at 224.155 131.445 180)
+      (effects (font (size 1.27 1.27)) (justify left))
+    )
+    (pin "I2C1_SCL" input (at 224.155 137.16 180)
+      (effects (font (size 1.27 1.27)) (justify left))
+    )
+    (pin "I2C1_SDA" input (at 224.155 140.97 180)
       (effects (font (size 1.27 1.27)) (justify left))
     )
@@
     )
   )
-  (sheet (at 159.385 29.845) (size 96.52 20.955)
+  (sheet (at 158.75 34.925) (size 96.52 20.955)
     (stroke (width 0.1524) (type solid))
     (fill (color 0 0 0 0.0000))
-    (property "Sheetname" "Capteur d'humidité, de pulsation, de température" (at 158.75 28.575 0)
+    (property "Sheetname" "Capteur d'humidité, de pulsation, de température" (at 158.115 33.655 0)
       (effects (font (size 2.54 2.54) bold (color 0 132 132 1)) (justify left bottom))
     )
-    (property "Sheetfile" "Capteur_humidite_pulsation_temperature.kicad_sch" (at 159.385 52.07 0)
+    (property "Sheetfile" "Capteur_humidite_pulsation_temperature.kicad_sch" (at 158.75 57.15 0)
       (effects (font (size 1.27 1.27)) (justify left top))
     )
-    (pin "Puls" output (at 255.905 34.925 0)
+    (pin "Puls" output (at 255.27 40.005 0)
       (effects (font (size 1.27 1.27)) (justify right))
     )
-    (pin "Temp" output (at 255.905 39.37 0)
+    (pin "Temp" output (at 255.27 44.45 0)
       (effects (font (size 1.27 1.27)) (justify right))
     )
-    (pin "Moist" output (at 255.905 43.815 0)
+    (pin "Moist" output (at 255.27 48.895 0)
       (effects (font (size 1.27 1.27)) (justify right))
     )
