File: ConceptionPCB_Projet_PAZ/Projet_PAZ/Trou_de_fixation.kicad_sch (KiCad schematic)
At the start: 4 parts

Commit message: Add files via upload
Parts:
- added H1, H11, H12, H13, H14, H15, H16, H17, H18, H3, H4, H6: MountingHole_Pad, MountingHole:MountingHole_2.5mm_Pad, symbol Mechanical:MountingHole_Pad
Connections:
- net GND: now also H1.1, H11.1, H12.1, H13.1, H14.1, H15.1, H16.1, H17.1, H18.1, H3.1, H4.1, H6.1
Other:
- moved on the sheet: H10, H2, H5, H9
